File: board/BarnDoorMount.sch (KiCad schematic (older format))
At the start: 33 parts, among them J1 SBW, J2 Shutter Control, J3 LCD, J4 Battery, J5 Stepper Motor, Q1 PZT2222A, Q2 PZT2222A, U1 MSP430FR2433, U2 LM317, U3 A3967

Commit message: Revision 2 of the driver board
Parts:
- added R16, R17, R18, R19, R20: 10K, Resistor_SMD:R_0603_1608Metric_Pad1.05x0.95mm_HandSolder, symbol Device:R_US
- added R21, R22: JUMPER, Resistor_SMD:R_0603_1608Metric_Pad1.05x0.95mm_HandSolder, symbol Device:R_US
- added R23: 390, Resistor_SMD:R_0603_1608Metric_Pad1.05x0.95mm_HandSolder, symbol Device:R_US
- added SW1: SELECT, Button_Switch_SMD:SW_SPST_B3S-1100, symbol Switch:SW_Push
- added SW2: OK, Button_Switch_SMD:SW_SPST_B3S-1100, symbol Switch:SW_Push
- added TP1: TP_GND, TestPoint:TestPoint_Pad_D2.0mm, symbol Connector:TestPoint
- added TP2: TP_33V, TestPoint:TestPoint_Pad_D2.0mm, symbol Connector:TestPoint
- J1: footprint Connector_PinHeader_2.54mm:PinHeader_1x02_P2.54mm_Vertical -> Connector_JST:JST_XH_B04B-XH-A_1x04_P2.50mm_Vertical; symbol Connector_Generic:Conn_01x02 -> Connector_Generic:Conn_01x04
- J2, J5: footprint Connector_PinHeader_2.54mm:PinHeader_1x04_P2.54mm_Vertical -> Connector_JST:JST_XH_B04B-XH-A_1x04_P2.50mm_Vertical
- J3: footprint Connector_PinHeader_2.54mm:PinHeader_1x08_P2.54mm_Vertical -> Connector_JST:JST_XH_S08B-XH-A_1x08_P2.50mm_Vertical
- J4: footprint Connector_PinHeader_2.54mm:PinHeader_1x02_P2.54mm_Vertical -> Connector_JST:JST_XH_B02B-XH-A_1x02_P2.50mm_Vertical
Connections:
- net labels added: OK_BTN, SELECT_BTN
- wire segments 116 -> 135
- no-connect marks 12 -> 8

Commit message: Board changes for rev 3: swap STEP and DIR pins between the MCU and stepper driver
Parts:
- J3: footprint Connector_JST:JST_XH_S08B-XH-A_1x08_P2.50mm_Vertical -> Connector_JST:JST_XH_B08B-XH-A_1x08_P2.50mm_Vertical
Connections:
- wire segments 135 -> 136
Changed lines of the file:
@@
 encoding utf-8
 Sheet 1 1
-Title "CameraMount"
+Title "Astrophotography Camera Controller"
 Date ""
-Rev "2"
-Comp ""
+Rev "3"
+Comp "csammis"
 Comment1 ""
 Comment2 ""
@@
 	8350 2800 8450 2800
 Connection ~ 8350 2800
-Wire Wire Line
-	5650 2000 6200 2000
 NoConn ~ 4400 2400
 NoConn ~ 4400 2500
@@
 F 0 "J3" V 5700 3350 50  0000 L CNN
 F 1 "LCD" V 5700 4000 50  0000 L CNN
-F 2 "Connector_JST:JST_XH_S08B-XH-A_1x08_P2.50mm_Vertical" H 5600 3800 50  0001 C CNN
+F 2 "Connector_JST:JST_XH_B08B-XH-A_1x08_P2.50mm_Vertical" H 5600 3800 50  0001 C CNN
 F 3 "~" H 5600 3800 50  0001 C CNN
 	1    5600 3800
@@
 	5650 1200 4400 1200
 Wire Wire Line
-	5650 1200 5650 2000
+	5650 1200 5650 1950
 Wire Wire Line
 	4400 1300 5550 1300
 Wire Wire Line
-	5550 1300 5550 2100
-Wire Wire Line
-	5550 2100 5950 2100
+	5550 1300 5550 2000
 NoConn ~ 4400 1900
 Text GLabel 4600 1400 2    50   Output ~ 0
@@
 L Device:R_US R16
 U 1 1 5BF8924F
-P 5950 2300
-F 0 "R16" H 6000 2350 50  0000 L CNN
-F 1 "10K" H 6000 2250 50  0000 L CNN
-F 2 "Resistor_SMD:R_0603_1608Metric_Pad1.05x0.95mm_HandSolder" V 5990 2290 50  0001 C CNN
-F 3 "~" H 5950 2300 50  0001 C CNN
-	1    5950 2300
+P 5550 2300
+F 0 "R16" H 5600 2350 50  0000 L CNN
+F 1 "10K" H 5600 2250 50  0000 L CNN
+F 2 "Resistor_SMD:R_0603_1608Metric_Pad1.05x0.95mm_HandSolder" V 5590 2290 50  0001 C CNN
+F 3 "~" H 5550 2300 50  0001 C CNN
+	1    5550 2300
 	1    0    0    -1
 $EndComp
@@
 L Device:R_US R17
 U 1 1 5BF892B7
-P 6200 2300
-F 0 "R17" H 6250 2350 50  0000 L CNN
-F 1 "10K" H 6250 2250 50  0000 L CNN
-F 2 "Resistor_SMD:R_0603_1608Metric_Pad1.05x0.95mm_HandSolder" V 6240 2290 50  0001 C CNN
-F 3 "~" H 6200 2300 50  0001 C CNN
-	1    6200 2300
-	1    0    0    -1
-$EndComp
-Wire Wire Line
-	6200 2000 6200 2150
-Wire Wire Line
-	5950 2100 5950 2150
+P 5850 2300
+F 0 "R17" H 5900 2350 50  0000 L CNN
+F 1 "10K" H 5900 2250 50  0000 L CNN
+F 2 "Resistor_SMD:R_0603_1608Metric_Pad1.05x0.95mm_HandSolder" V 5890 2290 50  0001 C CNN
+F 3 "~" H 5850 2300 50  0001 C CNN
+	1    5850 2300
+	1    0    0    -1
+$EndComp
 $Comp
 L power:GND #PWR027
 U 1 1 5BF9239E
-P 6200 2450
-F 0 "#PWR027" H 6200 2200 50  0001 C CNN
-F 1 "GND" H 6205 2277 50  0000 C CNN
-F 2 "" H 6200 2450 50  0001 C CNN
-F 3 "" H 6200 2450 50  0001 C CNN
-	1    6200 2450
+P 5850 2450
+F 0 "#PWR027" H 5850 2200 50  0001 C CNN
+F 1 "GND" H 5855 2277 50  0000 C CNN
+F 2 "" H 5850 2450 50  0001 C CNN
+F 3 "" H 5850 2450 50  0001 C CNN
+	1    5850 2450
 	1    0    0    -1
 $EndComp
@@
 L power:GND #PWR012
 U 1 1 5BF923F5
-P 5950 2450
-F 0 "#PWR012" H 5950 2200 50  0001 C CNN
-F 1 "GND" H 5955 2277 50  0000 C CNN
-F 2 "" H 5950 2450 50  0001 C CNN
-F 3 "" H 5950 2450 50  0001 C CNN
-	1    5950 2450
+P 5550 2450
+F 0 "#PWR012" H 5550 2200 50  0001 C CNN
+F 1 "GND" H 5555 2277 50  0000 C CNN
+F 2 "" H 5550 2450 50  0001 C CNN
+F 3 "" H 5550 2450 50  0001 C CNN
+	1    5550 2450
 	1    0    0    -1
 $EndComp
@@
 	1    0    0    -1
 $EndComp
-Connection ~ 5950 2100
-Connection ~ 6200 2000
-Wire Wire Line
-	6200 2000 7400 2000
-Wire Wire Line
-	5950 2100 7400 2100
 Wire Wire Line
 	6550 1750 6550 2200
@@
 Wire Wire Line
 	5200 3500 5200 3600
+Wire Wire Line
+	7050 2100 7400 2100
+Wire Wire Line
+	7050 1950 7050 2100
+Wire Wire Line
+	5850 1950 5850 2150
+Wire Wire Line
+	5550 2000 5550 2150
+Connection ~ 5550 2000
+Wire Wire Line
+	5550 2000 7400 2000
+Connection ~ 5850 1950
+Wire Wire Line
+	5850 1950 5650 1950
+Wire Wire Line
+	5850 1950 7050 1950
 $EndSCHEMATC
