File: board/AstroCameraAimer.sch (KiCad schematic (older format))
At the start: 45 parts, among them J1 SBW, J2 Shutter Control, J3 LCD, J4 Battery, J5 Stepper Motor, Q1 PZT2222A, Q2 PZT2222A, SW1 SELECT, SW2 OK, U1 MSP430FR2433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

Commit message: Updated schematic and PCB to revision 3
Parts:
- removed C5: 47uF, Capacitor_SMD:C_0805_2012Metric_Pad1.15x1.40mm_HandSolder, symbol Device:CP1_Small
- removed C6: 0.1uF, Capacitor_SMD:C_0603_1608Metric_Pad1.05x0.95mm_HandSolder, symbol Device:C_Small
- removed Q1, Q2: PZT2222A, Package_TO_SOT_SMD:SOT-223, symbol Transistor_BJT:PZT2222A
- removed R10, R23: 390, Resistor_SMD:R_0603_1608Metric_Pad1.05x0.95mm_HandSolder, symbol Device:R_US
- removed R14: 240, Resistor_SMD:R_0603_1608Metric_Pad1.05x0.95mm_HandSolder, symbol Device:R_US
- removed R16, R17, R18, R19, R20: 10K, Resistor_SMD:R_0603_1608Metric_Pad1.05x0.95mm_HandSolder, symbol Device:R_US
- removed R4, R5: 1K, Resistor_SMD:R_0603_1608Metric_Pad1.05x0.95mm_HandSolder, symbol Device:R_US
- removed SW1: SELECT, Button_Switch_SMD:SW_SPST_B3S-1100, symbol Switch:SW_Push
- removed SW2: OK, Button_Switch_SMD:SW_SPST_B3S-1100, symbol Switch:SW_Push
- removed U2: LM317, Package_TO_SOT_SMD:SOT-223-3_TabPin2, symbol Regulator_Linear:LM317_3PinPackage
- added C10: CL2, Capacitor_SMD:C_0603_1608Metric_Pad1.05x0.95mm_HandSolder, symbol Device:C_Small
- added C11, C12: 1uF, Capacitor_SMD:C_0603_1608Metric_Pad1.05x0.95mm_HandSolder, symbol Device:C_Small
- added C9: CL1, Capacitor_SMD:C_0603_1608Metric_Pad1.05x0.95mm_HandSolder, symbol Device:C_Small
- added H1, H2, H3: M2, MountingHole:MountingHole_2.2mm_M2, symbol Mechanical:MountingHole
- added J6: Buttons, Connector_JST:JST_XH_B03B-XH-A_1x03_P2.50mm_Vertical, symbol Connector_Generic:Conn_01x03
- added LG1: ProjectLogo, Logo:ursa_minor, symbol LocalGraphics:ProjectLogo
- added R2, R6: 100K, Resistor_SMD:R_0603_1608Metric_Pad1.05x0.95mm_HandSolder, symbol Device:R_Small_US
- added R5: 390, Resistor_SMD:R_0603_1608Metric_Pad1.05x0.95mm_HandSolder, symbol Device:R_Small_US
- added TP3: P3.0, TestPoint:TestPoint_Pad_D1.0mm, symbol Connector:TestPoint
- added TP4: P1.7, TestPoint:TestPoint_Pad_D1.0mm, symbol Connector:TestPoint
- added U2: ILD205, Package_SO:SOIC-8_3.9x4.9mm_P1.27mm, symbol LocalIsolator:ILD205
- added U4: NCP718, Package_TO_SOT_SMD:SOT-23-5_HandSoldering, symbol TransistorLocal:NCP718
- added U5: SiP32510, Package_TO_SOT_SMD:TSOT-23-6_HandSoldering, symbol LocalSwitches:SiP32510
- added Y1: 32Khz, Crystal:Crystal_SMD_MicroCrystal_CC7V-T1A-2Pin_3.2x1.5mm_HandSoldering, symbol Device:Crystal_Small
- J2: value Shutter Control -> Shutter; footprint Connector_JST:JST_XH_B04B-XH-A_1x04_P2.50mm_Vertical -> Connector_JST:JST_XH_B03B-XH-A_1x03_P2.50mm_Vertical; symbol Connector_Generic:Conn_01x04 -> Connector_Generic:Conn_01x03
- R1: symbol Device:R_US -> Device:R_Small_US
- R10: renamed from R8; value 10K -> 100K; symbol Device:R_US -> Device:R_Small_US
- R11: renamed from R9; value 6.8K -> 68K; symbol Device:R_US -> Device:R_Small_US
- R12: renamed from R21; symbol Device:R_US -> Device:R_Small_US
- R15: renamed from R11; symbol Device:R_US -> Device:R_Small_US
- R16: renamed from R12; value 0.75 -> 0.75Ω; symbol Device:R_US -> Device:R_Small_US
- R17: renamed from R13; value 0.75 -> 0.75Ω; symbol Device:R_US -> Device:R_Small_US
- R19: renamed from R22; symbol Device:R_US -> Device:R_Small_US
- R20: renamed from R15; symbol Device:R_US -> Device:R_Small_US
- R3: renamed from R2; value 10K -> 390; symbol Device:R_US -> Device:R_Small_US
- R4: renamed from R3; value 10K -> 390; symbol Device:R_US -> Device:R_Small_US
- R8: renamed from R7; symbol Device:R_US -> Device:R_Small_US
- R9: renamed from R6; symbol Device:R_US -> Device:R_Small_US
- TP1: value TP_GND -> GND; footprint TestPoint:TestPoint_Pad_D2.0mm -> TestPoint:TestPoint_Pad_D1.0mm
- TP2: value TP_33V -> 3.3V; footprint TestPoint:TestPoint_Pad_D2.0mm -> TestPoint:TestPoint_Pad_D1.0mm
Connections:
- net labels added: 9V, 9V_Coil1A, 9V_Coil1B, 9V_Coil2A, 9V_Coil2B, BATT_9V, DRIVER_DIR, DRIVER_STEP, DRIVER_nENABLE, DRIVER_nRESET, DRIVER_nSLEEP, LCD_CLK, LCD_DC, LCD_LED, LCD_MOSI, LCD_RST, LCD_nCS, SUPPLY_3.3V
- wire segments 136 -> 151
- no-connect marks 8 -> 0
Other:
- note added: "0.4 Vcc at PFD for mixed decay"
- note added: "Board markings"
- note added: "Display"
- note added: "Istepmax = Vref / (8 * Rsense) = 2V / 6Ω = 333mA"
- note added: "Optional"
- note added: "Power supply: Fixed LDO"
- note added: "Through-hole PCB mounts"

Commit message: Consolidating local symbol libraries
Parts:
- U1: symbol MSP430FR2433:MSP430FR2433 -> LocalICs:MSP430FR2433
- U3: symbol Allegro:A3967 -> LocalICs:A3967
- U4: symbol TransistorLocal:NCP718 -> LocalPower:NCP718
Changed lines of the file:
@@
 $EndDescr
 $Comp
-L MSP430FR2433:MSP430FR2433 U1
-U 1 1 5B6291B1
-P 1050 2750
-F 0 "U1" H 2756 4565 50  0000 C CNN
-F 1 "MSP430FR2433" H 2756 4474 50  0000 C CNN
-F 2 "Package_DFN_QFN:VQFN-24-1EP_4x4mm_P0.5mm_EP2.45x2.45mm" H 3150 4450 50  0001 C CNN
-F 3 "" H 1050 2750 50  0001 C CNN
-	1    1050 2750
-	1    0    0    -1
-$EndComp
-$Comp
-L Allegro:A3967 U3
+L LocalICs:A3967 U3
 U 1 1 5B679A45
 P 9600 2200
@@
 Text Label 7500 1550 0    39   ~ 0
 9V
-$Comp
-L TransistorLocal:NCP718 U4
-U 1 1 5CCC17DC
-P 8450 5750
-F 0 "U4" H 8300 5950 50  0000 L CNN
-F 1 "NCP718" H 8800 5950 50  0000 R CNN
-F 2 "Package_TO_SOT_SMD:SOT-23-5_HandSoldering" H 9300 5550 39  0001 C CNN
-F 3 "" H 8450 5750 39  0001 C CNN
-	1    8450 5750
-	1    0    0    -1
-$EndComp
 $Comp
 L power:GND #PWR0101
@@
 	0    -1   -1   0
 $EndComp
+$Comp
+L LocalICs:MSP430FR2433 U1
+U 1 1 5B6291B1
+P 1050 2750
+F 0 "U1" H 2756 4565 50  0000 C CNN
+F 1 "MSP430FR2433" H 2756 4474 50  0000 C CNN
+F 2 "Package_DFN_QFN:VQFN-24-1EP_4x4mm_P0.5mm_EP2.45x2.45mm" H 3150 4450 50  0001 C CNN
+F 3 "" H 1050 2750 50  0001 C CNN
+	1    1050 2750
+	1    0    0    -1
+$EndComp
+$Comp
+L LocalPower:NCP718 U4
+U 1 1 5CCC17DC
+P 8450 5750
+F 0 "U4" H 8300 5950 50  0000 L CNN
+F 1 "NCP718" H 8800 5950 50  0000 R CNN
+F 2 "Package_TO_SOT_SMD:SOT-23-5_HandSoldering" H 9300 5550 39  0001 C CNN
+F 3 "" H 8450 5750 39  0001 C CNN
+	1    8450 5750
+	1    0    0    -1
+$EndComp
 Wire Bus Line
-	4950 2800 4950 3400
+	4950 3000 4950 3300
 Wire Bus Line
-	4250 5875 4250 6275
+	4950 3300 4950 3400
+Wire Bus Line
+	4250 6075 4250 6175
+Wire Bus Line
+	4250 6175 4250 6275
+Wire Bus Line
+	4250 5975 4250 6075
+Wire Bus Line
+	4250 5875 4250 5975
+Wire Bus Line
+	4950 2900 4950 3000
+Wire Bus Line
+	4950 2800 4950 2900
 $EndSCHEMATC

Commit message: Fix NCP718 footprint and update board to revision 4
Changed lines of the file:
@@
 $EndComp
 Wire Bus Line
-	4950 3000 4950 3300
+	4950 2800 4950 3400
 Wire Bus Line
-	4950 3300 4950 3400
-Wire Bus Line
-	4250 6075 4250 6175
-Wire Bus Line
-	4250 6175 4250 6275
-Wire Bus Line
-	4250 5975 4250 6075
-Wire Bus Line
-	4250 5875 4250 5975
-Wire Bus Line
-	4950 2900 4950 3000
-Wire Bus Line
-	4950 2800 4950 2900
+	4250 5875 4250 6275
 $EndSCHEMATC
